File: Hardware/Qwiic EEPROM.sch (EAGLE design)
At the start: 29 parts, among them J3 PTH, U1 RM24C512C

Commit message: Add datasheet, make sure all parts are from SF libraries
Parts:
- removed J3: PTH, SparkX:I2C_STANDARD_NO_SILK
- removed U$1, U$2: SPARKX-LOGO4, SparkX:SPARKX-LOGO4
- added J5: (no value), SparkFun-Connectors:CONN_041X04_NO_SILK_NO_POP
- added JP7, JP8: STAND-OFF, SparkFun-Hardware:STAND-OFF
- added LOGO2: SFE_LOGO_NAME.2_INCH, SparkFun-Aesthetics:SFE_LOGO_NAME.2_INCH
- added LOGO3: SFE_LOGO_FLAME.2_INCH, SparkFun-Aesthetics:SFE_LOGO_FLAME.2_INCH
- added LOGO4: QWIIC_LOGO_3MM, SparkFun-Aesthetics:QWIIC_LOGO_3MM
- J2, J4: value (none) -> QWIIC_RA
- JP1, JP2, JP5, JP6: value FIDUCIALUFIDUCIAL -> FIDUCIAL0.2MM; device SparkFun:FIDUCIALUFIDUCIAL -> SparkFun-Aesthetics:FIDUCIAL0.2MM
- JP3, JP4: device SparkFun:STAND-OFF -> SparkFun-Hardware:STAND-OFF
- R4, R5: value 2.2k -> 4.7k; device SparkFun-Resistors:2.2KOHM-0603-1/10W-1% -> SparkFun-Resistors:4.7KOHM-0603-1/10W-1%
Connections:
- net 3.3V: now also J5.3; no longer J3.VCC
- net GND: now also J5.4; no longer J3.GND
- net SCL: now also J5.1; no longer J3.SCL
- net SDA: now also J5.2; no longer J3.SDA
Other:
- note added: "Connectors"
- note added: "EEPROM - 512Kbit"
- note added: "Power LED"
- note added: "Revised by: Priyanka Makin"
- note added: "v10"
- note removed: "X01"
- moved on the sheet: C4, D1, E0, E1, E2, I2C, J1, R1, R2, R3, R4, R5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

Commit message: Hardware updates
Schematic symbols from current SF libs
Added mounting holes
re-routing
Update 3.3V rail width
Parts:
- added POWER: JUMPER-SMT_2_NC_TRACE_SILK, SparkFun-Jumpers:JUMPER-SMT_2_NC_TRACE_SILK
Connections:
- new net N$10: D1.C, POWER.2
- net GND: now also POWER.1; no longer D1.C
Other:
- note removed: "Power"

Commit message: Vectorize labels
Parts:
- LOGO2: value SFE_LOGO_NAME.2_INCH -> SFE_LOGO_NAME.1_INCH; device SparkFun-Aesthetics:SFE_LOGO_NAME.2_INCH -> SparkFun-Aesthetics:SFE_LOGO_NAME.1_INCH
- LOGO3: value SFE_LOGO_FLAME.2_INCH -> SFE_LOGO_FLAME.1_INCH; device SparkFun-Aesthetics:SFE_LOGO_FLAME.2_INCH -> SparkFun-Aesthetics:SFE_LOGO_FLAME.1_INCH
- LOGO4: value QWIIC_LOGO_3MM -> QWIIC_LOGO_4MM; device SparkFun-Aesthetics:QWIIC_LOGO_3MM -> SparkFun-Aesthetics:QWIIC_LOGO_4MM
Changed lines of the file:
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@@
 <?xml version="1.0" encoding="utf-8"?>
 <!DOCTYPE eagle SYSTEM "eagle.dtd">
-<eagle version="9.5.2">
+<eagle version="9.6.2">
 <drawing>
 <settings>
@@
 <grid distance="0.1" unitdist="inch" unit="inch" style="lines" multiple="1" display="no" altdistance="0.01" altunitdist="inch" altunit="inch"/>
 <layers>
-<layer number="1" name="Top" color="4" fill="1" visible="no" active="no"/>
-<layer number="2" name="Route2" color="1" fill="3" visible="no" active="no"/>
-<layer number="3" name="Route3" color="4" fill="3" visible="no" active="no"/>
-<layer number="4" name="Route4" color="1" fill="4" visible="no" active="no"/>
-<layer number="5" name="Route5" color="4" fill="4" visible="no" active="no"/>
-<layer number="6" name="Route6" color="1" fill="8" visible="no" active="no"/>
-<layer number="7" name="Route7" color="4" fill="8" visible="no" active="no"/>
-<layer number="8" name="Route8" color="1" fill="2" visible="no" active="no"/>
-<layer number="9" name="Route9" color="4" fill="2" visible="no" active="no"/>
-<layer number="10" name="Route10" color="1" fill="7" visible="no" active="no"/>
-<layer number="11" name="Route11" color="4" fill="7" visible="no" active="no"/>
-<layer number="12" name="Route12" color="1" fill="5" visible="no" active="no"/>
-<layer number="13" name="Route13" color="4" fill="5" visible="no" active="no"/>
-<layer number="14" name="Route14" color="1" fill="6" visible="no" active="no"/>
-<layer number="15" name="Route15" color="4" fill="6" visible="no" active="no"/>
-<layer number="16" name="Bottom" color="1" fill="1" visible="no" active="no"/>
-<layer number="17" name="Pads" color="2" fill="1" visible="no" active="no"/>
-<layer number="18" name="Vias" color="2" fill="1" visible="no" active="no"/>
-<layer number="19" name="Unrouted" color="6" fill="1" visible="no" active="no"/>
-<layer number="20" name="Dimension" color="15" fill="1" visible="no" active="no"/>
-<layer number="21" name="tPlace" color="16" fill="1" visible="no" active="no"/>
-<layer number="22" name="bPlace" color="14" fill="1" visible="no" active="no"/>
-<layer number="23" name="tOrigins" color="15" fill="1" visible="no" active="no"/>
-<layer number="24" name="bOrigins" color="15" fill="1" visible="no" active="no"/>
-<layer number="25" name="tNames" color="7" fill="1" visible="no" active="no"/>
-<layer number="26" name="bNames" color="7" fill="1" visible="no" active="no"/>
-<layer number="27" name="tValues" color="7" fill="1" visible="no" active="no"/>
-<layer number="28" name="bValues" color="7" fill="1" visible="no" active="no"/>
+<layer number="1" name="Top" color="4" fill="1" visible="yes" active="no"/>
+<layer number="2" name="Route2" color="1" fill="3" visible="yes" active="no"/>
+<layer number="3" name="Route3" color="4" fill="3" visible="yes" active="no"/>
+<layer number="4" name="Route4" color="1" fill="4" visible="yes" active="no"/>
+<layer number="5" name="Route5" color="4" fill="4" visible="yes" active="no"/>
+<layer number="6" name="Route6" color="1" fill="8" visible="yes" active="no"/>
+<layer number="7" name="Route7" color="4" fill="8" visible="yes" active="no"/>
+<layer number="8" name="Route8" color="1" fill="2" visible="yes" active="no"/>
+<layer number="9" name="Route9" color="4" fill="2" visible="yes" active="no"/>
+<layer number="10" name="Route10" color="1" fill="7" visible="yes" active="no"/>
+<layer number="11" name="Route11" color="4" fill="7" visible="yes" active="no"/>
+<layer number="12" name="Route12" color="1" fill="5" visible="yes" active="no"/>
+<layer number="13" name="Route13" color="4" fill="5" visible="yes" active="no"/>
+<layer number="14" name="Route14" color="1" fill="6" visible="yes" active="no"/>
+<layer number="15" name="Route15" color="4" fill="6" visible="yes" active="no"/>
+<layer number="16" name="Bottom" color="1" fill="1" visible="yes" active="no"/>
+<layer number="17" name="Pads" color="2" fill="1" visible="yes" active="no"/>
+<layer number="18" name="Vias" color="2" fill="1" visible="yes" active="no"/>
+<layer number="19" name="Unrouted" color="6" fill="1" visible="yes" active="no"/>
+<layer number="20" name="Dimension" color="24" fill="1" visible="yes" active="no"/>
+<layer number="21" name="tPlace" color="16" fill="1" visible="yes" active="no"/>
+<layer number="22" name="bPlace" color="14" fill="1" visible="yes" active="no"/>
+<layer number="23" name="tOrigins" color="15" fill="1" visible="yes" active="no"/>
+<layer number="24" name="bOrigins" color="15" fill="1" visible="yes" active="no"/>
+<layer number="25" name="tNames" color="7" fill="1" visible="yes" active="no"/>
+<layer number="26" name="bNames" color="7" fill="1" visible="yes" active="no"/>
+<layer number="27" name="tValues" color="7" fill="1" visible="yes" active="no"/>
+<layer number="28" name="bValues" color="7" fill="1" visible="yes" active="no"/>
 <layer number="29" name="tStop" color="7" fill="3" visible="no" active="no"/>
 <layer number="30" name="bStop" color="7" fill="6" visible="no" active="no"/>
@@
 <layer number="35" name="tGlue" color="7" fill="4" visible="no" active="no"/>
 <layer number="36" name="bGlue" color="7" fill="5" visible="no" active="no"/>
-<layer number="37" name="tTest" color="7" fill="1" visible="no" active="no"/>
-<layer number="38" name="bTest" color="7" fill="1" visible="no" active="no"/>
+<layer number="37" name="tTest" color="7" fill="1" visible="yes" active="no"/>
+<layer number="38" name="bTest" color="7" fill="1" visible="yes" active="no"/>
 <layer number="39" name="tKeepout" color="4" fill="11" visible="no" active="no"/>
 <layer number="40" name="bKeepout" color="1" fill="11" visible="no" active="no"/>
@@
 <layer number="44" name="Drills" color="7" fill="1" visible="no" active="no"/>
 <layer number="45" name="Holes" color="7" fill="1" visible="no" active="no"/>
-<layer number="46" name="Milling" color="3" fill="1" visible="no" active="no"/>
-<layer number="47" name="Measures" color="7" fill="1" visible="no" active="no"/>
-<layer number="48" name="Document" color="7" fill="1" visible="no" active="no"/>
-<layer number="49" name="Reference" color="7" fill="1" visible="no" active="no"/>
-<layer number="50" name="dxf" color="7" fill="1" visible="no" active="no"/>
-<layer number="51" name="tDocu" color="6" fill="1" visible="no" active="no"/>
-<layer number="52" name="bDocu" color="7" fill="1" visible="no" active="no"/>
-<layer number="53" name="tGND_GNDA" color="7" fill="9" visible="no" active="no"/>
-<layer number="54" name="bGND_GNDA" color="1" fill="9" visible="no" active="no"/>
-<layer number="56" name="wert" color="7" fill="1" visible="no" active="no"/>
-<layer number="57" name="tCAD" color="7" fill="1" visible="no" active="no"/>
-<layer number="59" name="tCarbon" color="7" fill="1" visible="no" active="no"/>
-<layer number="60" name="bCarbon" color="7" fill="1" visible="no" active="no"/>
+<layer number="46" name="Milling" color="3" fill="1" visible="yes" active="no"/>
+<layer number="47" name="Measures" color="7" fill="1" visible="yes" active="no"/>
+<layer number="48" name="Document" color="7" fill="1" visible="yes" active="no"/>
+<layer number="49" name="Reference" color="7" fill="1" visible="yes" active="no"/>
+<layer number="50" name="dxf" color="7" fill="1" visible="yes" active="no"/>
+<layer number="51" name="tDocu" color="6" fill="1" visible="yes" active="no"/>
+<layer number="52" name="bDocu" color="7" fill="1" visible="yes" active="no"/>
+<layer number="53" name="tGND_GNDA" color="7" fill="9" visible="yes" active="no"/>
+<layer number="54" name="bGND_GNDA" color="1" fill="9" visible="yes" active="no"/>
+<layer number="56" name="wert" color="7" fill="1" visible="yes" active="no"/>
+<layer number="57" name="tCAD" color="7" fill="1" visible="yes" active="no"/>
+<layer number="59" name="tCarbon" color="7" fill="1" visible="yes" active="no"/>
+<layer number="60" name="bCarbon" color="7" fill="1" visible="yes" active="no"/>
 <layer number="88" name="SimResults" color="9" fill="1" visible="no" active="yes"/>
 <layer number="89" name="SimProbes" color="9" fill="1" visible="no" active="yes"/>
@@
 <part name="R6" library="SparkFun-Resistors" deviceset="10KOHM" device="-0603-1/10W-1%" value="10k"/>
 <part name="R7" library="SparkFun-Resistors" deviceset="10KOHM" device="-0603-1/10W-1%" value="10k"/>
-<part name="LOGO2" library="SparkFun-Aesthetics" deviceset="SFE_LOGO_NAME" device=".2_INCH"/>
+<part name="LOGO2" library="SparkFun-Aesthetics" deviceset="SFE_LOGO_NAME" device=".1_INCH" value="SFE_LOGO_NAME.1_INCH"/>
 <part name="JP7" library="SparkFun-Hardware" deviceset="STAND-OFF" device=""/>
 <part name="JP8" library="SparkFun-Hardware" deviceset="STAND-OFF" device=""/>
-<part name="LOGO3" library="SparkFun-Aesthetics" deviceset="SFE_LOGO_FLAME" device=".2_INCH"/>
-<part name="LOGO4" library="SparkFun-Aesthetics" deviceset="QWIIC_LOGO" device="_3MM"/>
+<part name="LOGO3" library="SparkFun-Aesthetics" deviceset="SFE_LOGO_FLAME" device=".1_INCH" value="SFE_LOGO_FLAME.1_INCH"/>
+<part name="LOGO4" library="SparkFun-Aesthetics" deviceset="QWIIC_LOGO" device="_4MM" value="QWIIC_LOGO_4MM"/>
 <part name="GND3" library="SparkFun-PowerSymbols" deviceset="GND" device=""/>
 <part name="J5" library="SparkFun-Connectors" deviceset="CONN_04" device="1X04_NO_SILK_NO_POP"/>

Commit message: Design review changes
Schematic:
* Added Vcc range for EEPROM IC
* Updated notes for power led and address jumpers
* Got rid of legacy font
* Replaced pullup/pulldown resistors R1, R2, R6, R7 to 100k

Board:
* Weird tRestrict on GND pad of EEPROM IC --> moved via around to avoid DRC errors
* Moved "PWR" label underneath the LED
* Moved "I2C" label so that it touches the silk of the jumper above it
* Re-routed 3.3V trace so that it does not run under the EEPROM IC
* Increased size of fiducials
* Made vias all the same size
* Added prod-id to the EEPROM IC
Parts:
- JP1, JP2, JP5, JP6: value FIDUCIAL0.2MM -> FIDUCIALUFIDUCIAL; device SparkFun-Aesthetics:FIDUCIAL0.2MM -> SparkFun-Aesthetics:FIDUCIALUFIDUCIAL
- R1, R2, R6, R7: value 10k -> 100k; device SparkFun-Resistors:10KOHM-0603-1/10W-1% -> SparkFun-Resistors:100KOHM-0603-1/10W-1%
- U1: PROD_ID (none) -> IC-14645
Other:
- note added: "Cut jumper to disable PWR LED."
- note added: "Cut jumper to remove I2C Pull-ups from bus"
- note added: "Vcc range: -0.3V to 3.6V"
- note removed: "Clear Jumper to remove I2C Pull-ups from bus"

Commit message: QC Double-check
Other:
- note added: "Max Vcc range: -0.3V to 3.6V"
- note removed: "Vcc range: -0.3V to 3.6V"
Changed lines of the file:
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@@
 <text x="63.5" y="177.8" size="2.54" layer="94" font="vector">EEPROM - 512Kbit</text>
 <text x="7.62" y="63.5" size="2.54" layer="94" font="vector">Connectors</text>
-<text x="132.08" y="78.74" size="1.778" layer="97" font="vector">Vcc range: -0.3V to 3.6V</text>
+<text x="127" y="81.28" size="1.778" layer="97" font="vector">Max Vcc range: -0.3V to 3.6V</text>
 <text x="27.94" y="124.46" size="1.778" layer="97" font="vector">Cut jumper to disable
 PWR LED.</text>

Commit message: Update EEPROM part number to CAT24C51 and re-generate schematic
Parts:
- U1: value RM24C512C -> CAT24C51
Changed lines of the file:
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@@
 <part name="SUPPLY10" library="SparkFun-PowerSymbols" deviceset="3.3V" device=""/>
 <part name="D1" library="SparkFun-LED" deviceset="LED-RED" device="0603" value="RED"/>
-<part name="U1" library="SparkFun-IC-Memory" deviceset="RM24C512C" device="">
+<part name="U1" library="SparkFun-IC-Memory" deviceset="RM24C512C" device="" value="CAT24C51">
 <attribute name="PROD_ID" value="IC-14645"/>
 </part>
